Commit message: fix:(changed dependecies and improved p-a-p-routine)

File: urdf/panda.urdf.xacro (robot description, xacro)
@@ -3,9 +3,9 @@
   <!-- === INCLUDE NECESSARY XACRO FILES === -->
   <xacro:include filename="$(find franka_description)/robots/common/franka_robot.xacro"/>
-  <xacro:include filename="$(find sp3_panda_ctrl)/urdf/traffic_light.urdf.xacro"/>
-  <xacro:include filename="$(find sp3_panda_ctrl)/urdf/table.urdf.xacro"/>
-  <xacro:include filename="$(find sp3_panda_ctrl)/urdf/lidar_sensor.urdf.xacro"/>
-  <xacro:include filename="$(find sp3_panda_ctrl)/urdf/realsense_d435.urdf.xacro"/>
-  <xacro:include filename="$(find sp3_panda_ctrl)/urdf/wall.urdf.xacro"/>
+  <xacro:include filename="$(find franka_description)/urdf/traffic_light.urdf.xacro"/>
+  <xacro:include filename="$(find franka_description)/urdf/table.urdf.xacro"/>
+  <xacro:include filename="$(find franka_description)/urdf/lidar_sensor.urdf.xacro"/>
+  <xacro:include filename="$(find franka_description)/urdf/realsense_d435.urdf.xacro"/>
+  <xacro:include filename="$(find franka_description)/urdf/wall.urdf.xacro"/>
   <xacro:arg name="arm_id" default="panda" />
   <!-- === FRANKA ROBOT === -->

File: urdf/realsense_d435.urdf.xacro (robot description, xacro)
@@ -8,6 +8,6 @@
 <robot name="sensor_d435" xmlns:xacro="http://ros.org/wiki/xacro">
   <!-- Includes -->
-  <xacro:include filename="$(find realsense2_description)/urdf/_materials.urdf.xacro" />
-  <xacro:include filename="$(find realsense2_description)/urdf/_usb_plug.urdf.xacro" />
+  <xacro:include filename="$(find franka_description)/urdf/_materials.urdf.xacro" />
+  <xacro:include filename="$(find franka_description)/urdf/_usb_plug.urdf.xacro" />
   <xacro:macro name="sensor_d435" params="parent *origin name:=camera use_nominal_extrinsics:=false add_plug:=false use_mesh:=true">
     <xacro:property name="M_PI" value="3.1415926535897931" />
@@ -53,5 +53,5 @@
           <origin xyz="${d435_zero_depth_to_glass + d435_glass_to_front} ${-d435_cam_depth_py} 0" rpy="${M_PI/2} 0 ${M_PI/2}"/>
           <geometry>
-            <mesh filename="package://realsense2_description/meshes/d435.dae" />
+            <mesh filename="package://sp3_panda_ctrl/meshes/d435.dae" />
           </geometry>
         </xacro:if>
